File: PT4115-Driver.brd (EAGLE design)
At the start: 26.5 x 35.6 mm, 21 parts, among them J1 M023.5MM

Commit message: Improved schematics and board aesthetics
Parts:
- C1, C2, C3: value (none) -> 22uF
- L1, L2, L3: value ELL6 -> 68uH
Other:
- board text added: "Francesco Truzzi www.truzzi.me"
- board text removed: "Francesco Truzzi - www.truzzi.me"
Changed lines of the file:
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@@
 <layer number="20" name="Dimension" color="15" fill="1" visible="yes" active="yes"/>
 <layer number="21" name="tPlace" color="7" fill="1" visible="yes" active="yes"/>
-<layer number="22" name="bPlace" color="7" fill="1" visible="no" active="yes"/>
+<layer number="22" name="bPlace" color="7" fill="1" visible="yes" active="yes"/>
 <layer number="23" name="tOrigins" color="15" fill="1" visible="yes" active="yes"/>
 <layer number="24" name="bOrigins" color="15" fill="1" visible="no" active="yes"/>
@@
 <text x="14.8" y="-1.4" size="1.016" layer="21" rot="R180">B</text>
 <text x="4.8" y="-2.4" size="1.016" layer="21">GND</text>
-<text x="21" y="-2" size="0.8128" layer="22" font="vector" rot="MR0">Francesco Truzzi - www.truzzi.me</text>
+<text x="10" y="7" size="1.4224" layer="22" font="vector" rot="MR0" align="center">Francesco Truzzi
+www.truzzi.me</text>
 <text x="10" y="24" size="1.778" layer="22" font="vector" rot="MR0" align="center">High power
 3-channel
@@
 <attribute name="VALUE" x="15.91" y="9.766" size="0.4064" layer="27"/>
 </element>
-<element name="L1" library="inductor-panasonic" package="ELL6" value="ELL6" x="1.56" y="21.56" smashed="yes">
+<element name="L1" library="inductor-panasonic" package="ELL6" value="68uH" x="1.56" y="21.56" smashed="yes">
 <attribute name="NAME" x="0.8025" y="21.035" size="1.016" layer="25" ratio="18"/>
 <attribute name="VALUE" x="-1.2975" y="17.4325" size="0.8128" layer="27" ratio="10"/>
 </element>
-<element name="L2" library="inductor-panasonic" package="ELL6" value="ELL6" x="9.962" y="21.56" smashed="yes">
+<element name="L2" library="inductor-panasonic" package="ELL6" value="68uH" x="9.962" y="21.56" smashed="yes">
 <attribute name="NAME" x="9.2045" y="21.035" size="1.016" layer="25" ratio="18"/>
 <attribute name="VALUE" x="7.1045" y="17.4325" size="0.8128" layer="27" ratio="10"/>
 </element>
-<element name="L3" library="inductor-panasonic" package="ELL6" value="ELL6" x="18.564" y="21.56" smashed="yes">
+<element name="L3" library="inductor-panasonic" package="ELL6" value="68uH" x="18.564" y="21.56" smashed="yes">
 <attribute name="NAME" x="17.9065" y="21.035" size="1.016" layer="25" ratio="18"/>
 <attribute name="VALUE" x="15.7065" y="17.4325" size="0.8128" layer="27" ratio="10"/>
@@
 <attribute name="VALUE" x="15.51" y="4.76" size="1.27" layer="27" rot="R180"/>
 </element>
-<element name="C1" library="rcl" package="D/7343-31R" value="" x="2" y="7" smashed="yes">
+<element name="C1" library="rcl" package="D/7343-31R" value="22uF" x="2" y="7" smashed="yes">
 <attribute name="NAME" x="1.25" y="7.6" size="0.8128" layer="25"/>
 <attribute name="VALUE" x="-1.65" y="3.425" size="1.27" layer="27"/>
 </element>
-<element name="C2" library="rcl" package="D/7343-31R" value="" x="12" y="7" smashed="yes">
+<element name="C2" library="rcl" package="D/7343-31R" value="22uF" x="12" y="7" smashed="yes">
 <attribute name="NAME" x="11.35" y="6.8" size="0.8128" layer="25"/>
 <attribute name="VALUE" x="8.35" y="3.425" size="1.27" layer="27"/>
 </element>
-<element name="C3" library="rcl" package="D/7343-31R" value="" x="20" y="6" smashed="yes" rot="R90">
+<element name="C3" library="rcl" package="D/7343-31R" value="22uF" x="20" y="6" smashed="yes" rot="R90">
 <attribute name="NAME" x="19.8" y="6.55" size="0.8128" layer="25" rot="R270"/>
 <attribute name="VALUE" x="23.575" y="2.35" size="1.27" layer="27" rot="R90"/>
